File: PICKit_Clone_KiCAD/PICKit_Clone_KiCAD.kicad_pcb (KiCad board)
At the start: 4 copper layers, 25 x 41.5 mm, 40 parts, among them J1 USB_C_Receptacle_USB2.0_16P, J2 Conn_02x03_Counter_Clockwise, Q1 MMBT3904, Q2 Si2319CDS, U1 PIC18F14K50-ESS, U2 MC34063AD, U3 LM1117MP-5.0, Y1 16MHz

Commit message: PCB and Design update
1) PCB has been modified to include pads for initial programming of the MCU
2)cover has been modified according to the new size of the PCB
Parts:
- added JP1: SolderJumper_2_Open, Jumper:SolderJumper-2_P1.3mm_Open_Pad1.0x1.5mm, F.Cu at (139.7, 83.4)
- added JP2: SolderJumper_2_Open, Jumper:SolderJumper-2_P1.3mm_Open_Pad1.0x1.5mm, F.Cu at (139.7, 86.2)
- added TP1: TestPoint, TestPoint:TestPoint_Pad_D1.0mm, F.Cu at (139.9, 111.5)
- added TP2: TestPoint, TestPoint:TestPoint_Pad_D1.0mm, F.Cu at (142.9, 111.5)
- added TP3: TestPoint, TestPoint:TestPoint_Pad_D1.0mm, F.Cu at (146.0, 111.5)
- added TP4: TestPoint, TestPoint:TestPoint_Pad_D1.0mm, F.Cu at (149.1, 111.5)
- added TP5: TestPoint, TestPoint:TestPoint_Pad_D1.0mm, F.Cu at (152.1, 111.5)
- Y1: value 16MHz -> Crystal_GND24; footprint Crystal:Crystal_SMD_HC49-SD -> Crystal:Crystal_SMD_3225-4Pin_3.2x2.5mm_HandSoldering
- moved C6 10.5 mm to (139.0, 89.0)
- moved Y1 5.81 mm to (138.7, 92.8), turned to 0 degrees
- moved C7 2.13 mm to (138.2, 96.7), turned to 0 degrees
Connections:
- U1 pad 4: unconnected-(U1-RA3/IOCA3/~{MCLR}/Vpp-Pad4) -> /mclr
- Y1 pad 2: Net-(U1-RA4/IOCA3/AN3/OSC2/CLKOUT) -> GND
Routing:
- net Net-(JP1-B): track 0.00 -> 32.8 mm
- net Net-(JP2-B): track 0.00 -> 31.4 mm
- net /mclr: track 0.00 -> 27.6 mm
- net Net-(U1-RA4/IOCA3/AN3/OSC2/CLKOUT): track 17.4 -> 8.83 mm
- net /USB_DP: track 11.7 -> 17.1 mm
- net /USB_DN: track 11.6 -> 16.9 mm
- net GND: vias 19 -> 22
- net /5V: vias 9 -> 10
Other:
- board size 25 x 41.5 mm -> 25 x 43 mm
